File: Hardware/Regenerative_Braking/MCU_peripherals.kicad_sch (KiCad schematic)
At the start: 0 parts

Commit message: Added Battery side
Parts:
- added U1: NUCLEO-F446RE, NUCLEO-F446RE:MODULE_NUCLEO-F446RE, symbol Regen_braking:NUCLEO-F446RE
Connections:
- new net CN7_GND: U1.CN7_19 (CN7_GND), U1.CN7_20 (CN7_GND), U1.CN7_22 (CN7_GND), U1.CN7_8 (CN7_GND)

Commit message: finished everything except mcu
Other:
- moved on the sheet: U1A
Changed lines of the file:
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@@
 	(symbol
 		(lib_id "Regen_braking:NUCLEO-F446RE")
-		(at 134.62 110.49 0)
+		(at 143.51 88.9 0)
 		(unit 1)
 		(body_style 1)
@@
 		(fields_autoplaced yes)
 		(property "Reference" "U1"
-			(at 134.62 64.77 0)
+			(at 143.51 43.18 0)
 			(show_name no)
 			(do_not_autoplace no)
@@
 		)
 		(property "Value" "NUCLEO-F446RE"
-			(at 134.62 67.31 0)
+			(at 143.51 45.72 0)
 			(show_name no)
 			(do_not_autoplace no)
@@
 		)
 		(property "Footprint" "NUCLEO-F446RE:MODULE_NUCLEO-F446RE"
-			(at 134.62 110.49 0)
+			(at 143.51 88.9 0)
 			(hide yes)
 			(show_name no)
@@
 		)
 		(property "Datasheet" ""
-			(at 134.62 110.49 0)
+			(at 143.51 88.9 0)
 			(hide yes)
 			(show_name no)
@@
 		)
 		(property "Description" "STM32F446RE, mbed-Enabled Development Nucleo-64 STM32F4 ARM® Cortex®-M4 MCU 32-Bit Embedded Evaluation Board"
-			(at 134.62 110.49 0)
+			(at 143.51 88.9 0)
 			(hide yes)
 			(show_name no)
@@
 		)
 		(property "MF" "STMicroelectronics"
-			(at 134.62 110.49 0)
+			(at 143.51 88.9 0)
 			(hide yes)
 			(show_name no)
@@
 		)
 		(property "MAXIMUM_PACKAGE_HEIGHT" ""
-			(at 134.62 110.49 0)
+			(at 143.51 88.9 0)
 			(hide yes)
 			(show_name no)
@@
 		)
 		(property "Package" "None"
-			(at 134.62 110.49 0)
+			(at 143.51 88.9 0)
 			(hide yes)
 			(show_name no)
@@
 		)
 		(property "Price" "None"
-			(at 134.62 110.49 0)
+			(at 143.51 88.9 0)
 			(hide yes)
 			(show_name no)
@@
 		)
 		(property "Check_prices" "https://www.snapeda.com/parts/NUCLEO-F446RE/STMicroelectronics/view-part/?ref=eda"
-			(at 134.62 110.49 0)
+			(at 143.51 88.9 0)
 			(hide yes)
 			(show_name no)
@@
 		)
 		(property "STANDARD" "Manufacturer Recommendations"
-			(at 134.62 110.49 0)
+			(at 143.51 88.9 0)
 			(hide yes)
 			(show_name no)
@@
 		)
 		(property "PARTREV" "13"
-			(at 134.62 110.49 0)
+			(at 143.51 88.9 0)
 			(hide yes)
 			(show_name no)
@@
 		)
 		(property "SnapEDA_Link" "https://www.snapeda.com/parts/NUCLEO-F446RE/STMicroelectronics/view-part/?ref=snap"
-			(at 134.62 110.49 0)
+			(at 143.51 88.9 0)
 			(hide yes)
 			(show_name no)
@@
 		)
 		(property "MP" "NUCLEO-F446RE"
-			(at 134.62 110.49 0)
+			(at 143.51 88.9 0)
 			(hide yes)
 			(show_name no)
@@
 		)
 		(property "Purchase-URL" "https://www.snapeda.com/api/url_track_click_mouser/?unipart_id=284290&manufacturer=STMicroelectronics&part_name=NUCLEO-F446RE&search_term=stm32 nucleo-64 development board with stm32f446re mcu"
-			(at 134.62 110.49 0)
+			(at 143.51 88.9 0)
 			(hide yes)
 			(show_name no)
@@
 		)
 		(property "Availability" "In Stock"
-			(at 134.62 110.49 0)
+			(at 143.51 88.9 0)
 			(hide yes)
 			(show_name no)
@@
 		)
 		(property "MANUFACTURER" "STMicroelectronics"
-			(at 134.62 110.49 0)
-			(hide yes)
-			(show_name no)
+			(at 143.51 88.9 0)
+			(hide yes)
+			(show_name no)

Commit message: MCU CONNECTIONS
Parts:
- added unit 6 of U1
- added unit 4 of U1
- added unit 5 of U1
- added unit 2 of U1
- added unit 3 of U1
- U1: footprint NUCLEO-F446RE:MODULE_NUCLEO-F446RE -> Regen_braking:MODULE_NUCLEO-F446RE
Connections:
- net U_ADC1: now reaches U1.CN7_28 (PA0)
- net VSENSE_BAT: now reaches U1.CN7_30 (PA1)
- net V_ADC1: now reaches U1.CN7_32 (PA4)
- net W_ADC1: now reaches U1.CN7_34 (PB0)
- net OUT3: now reaches U1.CN7_38 (PC0/PB8)
- net GND: now reaches U1.CN7_7 (BOOT0)
- new net CN10_GND: U1.CN10_20 (CN10_GND), U1.CN10_9 (CN10_GND)
- new net CN6_GND: U1.CN6_6 (CN6_GND), U1.CN6_7 (CN6_GND)
- new net OUT1: U1.CN10_15 (PA7)
- new net OUT2: U1.CN10_24 (PB1)
- new net OUT4: U1.CN10_13 (PA6), U1.CN10_22 (PB2)
- new net RX: U1.CN10_37 (PA3)
- new net TX: U1.CN10_35 (PA2)
- new net U_HIGH: U1.CN10_23 (PA8)
- new net U_LOW: U1.CN10_30 (PB13)
- new net V_HIGH: U1.CN10_21 (PA9)
- new net V_LOW: U1.CN10_28 (PB14)
- new net W_HIGH: U1.CN10_33 (PA10)
- new net W_LOW: U1.CN10_26 (PB15)
Other:
- moved on the sheet: U1A

Commit message: finished schematic
Parts:
- U1: footprint NUCLEO-F446RE:MODULE_NUCLEO-F446RE -> Regen_braking:MODULE_NUCLEO-F446RE
Connections:
- net OUT4: now also U1.CN10_16 (PB12); no longer U1.CN10_22 (PB2)
- net Hall_V: now reaches U1.CN10_19 (PC7)
- net Hall_W: now reaches U1.CN10_2 (PC8)
- net Hall_U: now reaches U1.CN10_4 (PC6)
- net ACS2: now reaches U1.CN7_35 (PC2)
- net ACS1: now reaches U1.CN7_36 (PC1/PB9)
- net VSENSE_CAP: now reaches U1.CN7_37 (PC3)
Changed lines of the file:
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@@
+	(wire
+		(pts
+			(xy 27.94 105.41) (xy 34.29 105.41)
+		)
+		(stroke
+			(width 0)
+			(type default)
+		)
+	)
 	(wire
 		(pts
@@
 	(wire
 		(pts
-			(xy 114.3 82.55) (xy 118.11 82.55)
+			(xy 114.3 69.85) (xy 118.11 69.85)
 		)
 		(stroke
@@
 	(wire
 		(pts
-			(xy 114.3 69.85) (xy 118.11 69.85)
+			(xy 153.67 64.77) (xy 157.48 64.77)
 		)
 		(stroke
@@
 	(wire
 		(pts
-			(xy 114.3 80.01) (xy 118.11 80.01)
+			(xy 27.94 110.49) (xy 34.29 110.49)
 		)
 		(stroke
@@
 	(wire
 		(pts
-			(xy 114.3 59.69) (xy 118.11 59.69)
+			(xy 153.67 67.31) (xy 157.48 67.31)
 		)
 		(stroke
@@
 	(wire
 		(pts
-			(xy 27.94 102.87) (xy 34.29 102.87)
+			(xy 114.3 59.69) (xy 118.11 59.69)
 		)
 		(stroke
@@
 	(wire
 		(pts
-			(xy 114.3 74.93) (xy 118.11 74.93)
+			(xy 153.67 69.85) (xy 157.48 69.85)
 		)
 		(stroke
@@
 	(wire
 		(pts
-			(xy 113.03 115.57) (xy 118.11 115.57)
+			(xy 113.03 110.49) (xy 118.11 110.49)
 		)
 		(stroke
@@
 	(wire
 		(pts
-			(xy 27.94 72.39) (xy 34.29 72.39)
+			(xy 27.94 102.87) (xy 34.29 102.87)
 		)
 		(stroke
@@
 	(wire
 		(pts
-			(xy 27.94 77.47) (xy 34.29 77.47)
+			(xy 114.3 74.93) (xy 118.11 74.93)
 		)
 		(stroke
@@
 	(wire
 		(pts
-			(xy 114.3 90.17) (xy 118.11 90.17)
+			(xy 113.03 115.57) (xy 118.11 115.57)
+		)
+		(stroke
+			(width 0)
+			(type default)
+		)
+	)
+	(wire
+		(pts
+			(xy 27.94 72.39) (xy 34.29 72.39)
+		)
+		(stroke
+			(width 0)
+			(type default)
+		)
+	)
+	(wire
+		(pts
+			(xy 27.94 77.47) (xy 34.29 77.47)
+		)
+		(stroke
+			(width 0)
+			(type default)
+		)
+	)
+	(wire
+		(pts
+			(xy 27.94 107.95) (xy 34.29 107.95)
 		)
 		(stroke
@@
 		)
 	)
+	(label "ACS2"
+		(at 27.94 107.95 180)
+		(effects
+			(font
+				(size 1.27 1.27)
+			)
+			(justify right bottom)
+		)
+	)
 	(label "V_HIGH"
 		(at 114.3 74.93 180)
@@
 		)
 	)
+	(label "Hall_W"
+		(at 157.48 69.85 0)
+		(effects
+			(font
+				(size 1.27 1.27)
+			)
+			(justify left bottom)
+		)
+	)
 	(label "W_HIGH"
 		(at 114.3 77.47 180)
@@
 		)
 	)
+	(label "Hall_U"
+		(at 157.48 64.77 0)
+		(effects
+			(font
+				(size 1.27 1.27)
+			)
+			(justify left bottom)
+		)
+	)
 	(label "V_LOW"
 		(at 113.03 115.57 180)
@@
 	)
 	(label "OUT4"
-		(at 114.3 90.17 180)
+		(at 113.03 110.49 180)
 		(effects
 			(font
@@
 		)
 	)
+	(label "ACS1"
+		(at 27.94 105.41 180)
+		(effects
+			(font
+				(size 1.27 1.27)
+			)
+			(justify right bottom)
+		)
+	)
 	(label "W_ADC1"
 		(at 27.94 95.25 180)
@@
 			)
 			(justify right bottom)
+		)
+	)
+	(label "VSENSE_CAP"
+		(at 27.94 110.49 180)
+		(effects
+			(font
+				(size 1.27 1.27)
+			)
+			(justify right bottom)
+		)
+	)
+	(label "Hall_V"
+		(at 157.48 67.31 0)
+		(effects
+			(font
+				(size 1.27 1.27)
+			)
+			(justify left bottom)
 		)
 	)
@@
 			)
 		)
-		(property "Footprint" "NUCLEO-F446RE:MODULE_NUCLEO-F446RE"
+		(property "Footprint" "Regen_braking:MODULE_NUCLEO-F446RE"
 			(at 260.35 52.07 0)
 			(hide yes)
@@
 			)
 		)
-		(property "Footprint" "NUCLEO-F446RE:MODULE_NUCLEO-F446RE"
+		(property "Footprint" "Regen_braking:MODULE_NUCLEO-F446RE"
 			(at 204.47 119.38 0)
 			(hide yes)
@@
 			)
 		)
-		(property "Footprint" "NUCLEO-F446RE:MODULE_NUCLEO-F446RE"
+		(property "Footprint" "Regen_braking:MODULE_NUCLEO-F446RE"
 			(at 203.2 53.34 0)
 			(hide yes)
@@
 			)
 		)
-		(property "Footprint" "NUCLEO-F446RE:MODULE_NUCLEO-F446RE"
+		(property "Footprint" "Regen_braking:MODULE_NUCLEO-F446RE"
 			(at 135.89 87.63 0)
 			(hide yes)
@@
 			)
 		)
-		(property "Footprint" "NUCLEO-F446RE:MODULE_NUCLEO-F446RE"
+		(property "Footprint" "Regen_braking:MODULE_NUCLEO-F446RE"
 			(at 259.08 116.84 0)
 			(hide yes)

Commit message: finished placement
Parts:
- removed U1: NUCLEO-F446RE, Regen_braking:MODULE_NUCLEO-F446RE, symbol Regen_braking:NUCLEO-F446RE
- added D10, D7, D8, D9: LED, LED_THT:LED_D5.0mm, symbol Device:LED
- added J10, J5, J6: Conn_01x06, Connector_PinHeader_2.54mm:PinHeader_1x06_P2.54mm_Vertical, symbol Connector_Generic:Conn_01x06
- added J11, J24, J25, J26: Conn_01x02, Connector_PinHeader_2.54mm:PinHeader_1x02_P2.54mm_Vertical, symbol Connector_Generic:Conn_01x02
- added J12, J27, J28, J29, J30, J31, J32: Conn_01x01, Connector_PinHeader_2.54mm:PinHeader_1x01_P2.54mm_Vertical, symbol Connector_Generic:Conn_01x01
- added J7: Conn_01x10, Connector_PinHeader_2.54mm:PinHeader_1x10_P2.54mm_Vertical, symbol Connector_Generic:Conn_01x10
- added J8: Conn_01x04, Connector_PinHeader_2.54mm:PinHeader_1x04_P2.54mm_Vertical, symbol Connector_Generic:Conn_01x04
- added J9: Conn_01x03, Connector_PinHeader_2.54mm:PinHeader_1x03_P2.54mm_Vertical, symbol Connector_Generic:Conn_01x03
- added R12, R13, R14, R15: 22, Resistor_THT:R_Axial_DIN0204_L3.6mm_D1.6mm_P7.62mm_Horizontal, symbol Device:R
Connections:
- net ACS1: now also J31.1 (Pin_1)
- net ACS2: now also J32.1 (Pin_1)
- net GND: now also D10.1 (K), D7.1 (K), D8.1 (K), D9.1 (K), J7.1 (Pin_1), J7.10 (Pin_10), J7.2 (Pin_2), J7.3 (Pin_3), J7.4 (Pin_4), J7.5 (Pin_5), J7.6 (Pin_6), J7.7 (Pin_7), J7.8 (Pin_8), J7.9 (Pin_9)
- net Hall_U: now also J9.1 (Pin_1)
- net Hall_V: now also J9.2 (Pin_2)
- net Hall_W: now also J9.3 (Pin_3)
- net OUT1: now also J10.1 (Pin_1)
- net OUT2: now also J10.2 (Pin_2)
- net OUT3: now also J10.3 (Pin_3)
- net OUT4: now also J10.4 (Pin_4), J10.5 (Pin_5), J10.6 (Pin_6)
- net U_ADC1: now also J12.1 (Pin_1)
- net U_HIGH: now also J11.1 (Pin_1)
- net U_LOW: now also J11.2 (Pin_2)
- net VSENSE_BAT: now also J29.1 (Pin_1)
- net VSENSE_CAP: now also J30.1 (Pin_1)
- net V_ADC1: now also J27.1 (Pin_1)
- net V_HIGH: now also J24.2 (Pin_2)
- net V_LOW: now also J24.1 (Pin_1)
- net W_ADC1: now also J28.1 (Pin_1)
- net W_HIGH: now also J25.1 (Pin_1)
- net W_LOW: now also J25.2 (Pin_2)
- new net: D9.2 (A), R14.1
- new net: J8.3 (Pin_3), R14.2
- new net: J6.1 (Pin_1), J6.2 (Pin_2), J6.3 (Pin_3), J6.4 (Pin_4), J6.5 (Pin_5), J6.6 (Pin_6)
- new net: J8.1 (Pin_1), R12.2
- new net: J8.2 (Pin_2), R13.2
- new net: J8.4 (Pin_4), R15.2
- new net: D8.2 (A), R13.1
- new net: D7.2 (A), R12.1
- new net: J5.1 (Pin_1), J5.2 (Pin_2), J5.3 (Pin_3), J5.4 (Pin_4), J5.5 (Pin_5), J5.6 (Pin_6)
- new net: D10.2 (A), R15.1
- new net Q_HIGH: J26.1 (Pin_1)
- new net Q_LOW: J26.2 (Pin_2)
- no-connect marks 0 -> 2
Other:
- note added: "3V3 PORTS"
- note added: "5V PORTS"
- note added: "ADC PORTS"
- note added: "COMP-EXTI BLOCK"
- note added: "GND PORTS"
- note added: "GPIO BLOCK"
- note added: "HALL-EXTI BLOCK"
- note added: "PWM PORTS"

Commit message: ------------------Project Completed Successfully------------------
Parts:
- removed J31, J32: Conn_01x01, Connector_PinHeader_2.54mm:PinHeader_1x01_P2.54mm_Vertical, symbol Connector_Generic:Conn_01x01
- added J21: ACS1_ADC, Connector_PinHeader_2.54mm:PinHeader_1x01_P2.54mm_Vertical, symbol Connector_Generic:Conn_01x01
- J10: value Conn_01x06 -> COMP_EXTI
- J11: value Conn_01x02 -> U_PWM
- J12: value Conn_01x01 -> U_ADC
- J24: value Conn_01x02 -> V_PWM
- J25: value Conn_01x02 -> W_PWM
- J26: value Conn_01x02 -> Q_PWM
- J27: value Conn_01x01 -> V_ADC
- J28: value Conn_01x01 -> W_ADC
- J29: value Conn_01x01 -> BAT_ADC
- J30: value Conn_01x01 -> CAP_ADC
- J5: value Conn_01x06 -> 3V3_ports
- J6: value Conn_01x06 -> 5V_ports
- J7: value Conn_01x10 -> GND_ports
- J8: value Conn_01x04 -> GPIO_ports
- J9: value Conn_01x03 -> HALL_EXTI
Connections:
- net ACS1: now also J21.1 (Pin_1)
