File: Hardware/Regenerative_Braking/Regenerative_Braking.kicad_pcb (KiCad board)
At the start: 2 copper layers, 39 parts, among them IC1 IRS21867STRPBF, IC2 IRS21867STRPBF, IC3 IRS21867STRPBF

Commit message: finished placement
Parts:
- removed R_ON_10ohm1, R_ON_10ohm2, R_ON_10ohm3, R_ON_10ohm4, R_ON_10ohm5, R_ON_10ohm6: ~, Regen_braking:R_ON_10ohm
- added C10: 1000uf, Capacitor_THT:C_Radial_D12.5mm_H25.0mm_P5.00mm, F.Cu at (225.2, 155.1)
- added C11: 1000uf, Capacitor_THT:C_Radial_D12.5mm_H25.0mm_P5.00mm, F.Cu at (212.1, 155.1)
- added C12: 1000uf, Capacitor_THT:C_Radial_D12.5mm_H25.0mm_P5.00mm, F.Cu at (199.1, 155.1)
- added C13: 1000uf, Capacitor_THT:C_Radial_D12.5mm_H25.0mm_P5.00mm, F.Cu at (186.0, 155.1)
- added C14: 1000uf, Capacitor_THT:C_Radial_D12.5mm_H25.0mm_P5.00mm, F.Cu at (172.9, 155.1)
- added C15: 0.47uf_50v_BScap, Regen_braking:0.47uf_50v_BScap, B.Cu at (143.3, 94.0)
- added C16: 1nf_snubber, Capacitor_SMD:C_1206_3216Metric, B.Cu at (169.1, 92.2)
- added C17: 4.7uf_50v_VDDcap, Regen_braking:4.7uf_50v_VDDcap, B.Cu at (155.3, 94.5)
- added C18: 1nf_snubber, Capacitor_SMD:C_1206_3216Metric, B.Cu at (169.1, 106.5)
- added C19: 0.47uf_50v_BScap, Regen_braking:0.47uf_50v_BScap, B.Cu at (172.7, 94.1)
- added C20: 33p, Capacitor_SMD:C_0805_2012Metric, F.Cu at (26.4, 158.7)
- added C21: 1nf_snubber, Capacitor_SMD:C_1206_3216Metric, B.Cu at (198.1, 92.0)
- added C22: 4.7uf_50v_VDDcap, Regen_braking:4.7uf_50v_VDDcap, B.Cu at (184.7, 94.7)
- added C23: 33p, Capacitor_SMD:C_0805_2012Metric, F.Cu at (29.4, 158.7)
- added C24: 1nf_snubber, Capacitor_SMD:C_1206_3216Metric, B.Cu at (198.2, 106.4)
- added C25: 1nf_snubber, Capacitor_SMD:C_1206_3216Metric, B.Cu at (225.0, 92.0)
- added C26: 33p, Capacitor_SMD:C_0805_2012Metric, F.Cu at (26.4, 166.9)
- added C27: 0.47uf_50v_BScap, Regen_braking:0.47uf_50v_BScap, B.Cu at (202.0, 93.9)
- added C28: 4.7uf_50v_VDDcap, Regen_braking:4.7uf_50v_VDDcap, B.Cu at (214.0, 94.6)
- added C29: 33p, Capacitor_SMD:C_0805_2012Metric, F.Cu at (29.4, 166.9)
- added C30: 1nf_snubber, Capacitor_SMD:C_1206_3216Metric, B.Cu at (225.0, 106.4)
- added C31: 33p, Capacitor_SMD:C_0805_2012Metric, F.Cu at (26.4, 174.9)
- added C32: 0.47uf_50v_BScap, Regen_braking:0.47uf_50v_BScap, B.Cu at (227.4, 94.1)
- added C33: 1nf_snubber, Capacitor_SMD:C_1206_3216Metric, B.Cu at (252.4, 91.9)
- added C34: 4.7uf_50v_VDDcap, Regen_braking:4.7uf_50v_VDDcap, B.Cu at (239.4, 94.7)
- added C35: 33p, Capacitor_SMD:C_0805_2012Metric, F.Cu at (29.4, 174.9)
- added C36: 1nf_snubber, Capacitor_SMD:C_1206_3216Metric, B.Cu at (252.3, 106.4)
- added C37: 10nf_rcFilter, Capacitor_THT:C_Disc_D6.0mm_W4.4mm_P5.00mm, F.Cu at (239.9, 138.4)
- added C38: 10nf_rcFilter, Capacitor_THT:C_Disc_D6.0mm_W4.4mm_P5.00mm, F.Cu at (184.5, 127.9)
- added C39: 100nf_rcFilter, Capacitor_SMD:C_1206_3216Metric, F.Cu at (178.0, 45.4)
- added C40: 10nf_rcFilter, Capacitor_THT:C_Disc_D6.0mm_W4.4mm_P5.00mm, F.Cu at (251.3, 138.5)
- added C41: 100nf_rcFilter, Capacitor_SMD:C_1206_3216Metric, F.Cu at (148.4, 155.2)
- added C42: 10nf_rcFilter, Capacitor_THT:C_Disc_D6.0mm_W4.4mm_P5.00mm, F.Cu at (217.0, 128.0)
- added C43: 10nf_rcFilter, Capacitor_THT:C_Disc_D6.0mm_W4.4mm_P5.00mm, F.Cu at (262.5, 138.5)
- added C44: 10nf_rcFilter, Capacitor_THT:C_Disc_D6.0mm_W4.4mm_P5.00mm, F.Cu at (249.3, 128.0)
- added C45: 100nf_rcFilter, Capacitor_SMD:C_1206_3216Metric, F.Cu at (197.8, 164.6)
- added C46: 100nf_rcFilter, Capacitor_SMD:C_1206_3216Metric, F.Cu at (155.8, 148.2)
- added C47: 100nf_rcFilter, Capacitor_SMD:C_1206_3216Metric, F.Cu at (212.0, 45.0)
- added C7: 1000uf, Capacitor_THT:C_Radial_D12.5mm_H25.0mm_P5.00mm, F.Cu at (212.1, 136.9)
- added C8: 1000uf, Capacitor_THT:C_Radial_D12.5mm_H25.0mm_P5.00mm, F.Cu at (225.2, 136.9)
- added C9: 330uf, Regen_braking:330uf_25v_cap_5v_buck, F.Cu at (166.2, 52.5)
- added C_Hi1: 33p, Capacitor_SMD:C_0805_2012Metric, F.Cu at (26.4, 182.0)
- added C_Li1: 33p, Capacitor_SMD:C_0805_2012Metric, F.Cu at (29.4, 182.0)
- added D10: LED, LED_THT:LED_D5.0mm, F.Cu at (51.3, 28.2)
- added D11: D_boot, Regen_braking:boot_diode, B.Cu at (185.9, 103.0)
- added D12: SS34_UH, Regen_braking:DIO_SS34, B.Cu at (178.7, 87.7)
- added D13: SS34_UL, Regen_braking:DIO_SS34, B.Cu at (178.4, 112.2)
- added D14: D_boot, Regen_braking:boot_diode, B.Cu at (213.1, 103.3)
- added D15: SS34_VH, Regen_braking:DIO_SS34, B.Cu at (208.0, 87.7)
- added D16: SS34_VL, Regen_braking:DIO_SS34, B.Cu at (205.5, 112.3)
- added D17: D_boot, Regen_braking:boot_diode, B.Cu at (239.8, 102.9)
- added D18: SS34_WH, Regen_braking:DIO_SS34, B.Cu at (233.3, 87.8)
- added D19: SS34_WL, Regen_braking:DIO_SS34, B.Cu at (232.0, 112.4)
- added D_OV1: BAT54T1G, Regen_braking:SODFL3718X115, F.Cu at (173.5, 45.4)
- added D_OV2: BAT54T1G, Regen_braking:SODFL3718X115, F.Cu at (178.7, 124.6)
- added D_OV3: BAT54T1G, Regen_braking:SODFL3718X115, F.Cu at (211.3, 124.7)
- added D_OV4: BAT54T1G, Regen_braking:SODFL3718X115, F.Cu at (243.6, 125.0)
- added D_OV5: BAT54T1G, Regen_braking:SODFL3718X115, F.Cu at (202.3, 164.4)
- added D_OV6: BAT54T1G, Regen_braking:SODFL3718X115, F.Cu at (160.4, 148.2)
- added D_OV7: BAT54T1G, Regen_braking:SODFL3718X115, F.Cu at (207.5, 45.0)
- added D_UV1: BAT54T1G, Regen_braking:SODFL3718X115, F.Cu at (180.9, 125.6)
- added D_UV2: BAT54T1G, Regen_braking:SODFL3718X115, F.Cu at (175.7, 45.6)
- added D_UV3: BAT54T1G, Regen_braking:SODFL3718X115, F.Cu at (213.4, 125.8)
- added D_UV4: BAT54T1G, Regen_braking:SODFL3718X115, F.Cu at (245.7, 126.0)
- added D_UV5: BAT54T1G, Regen_braking:SODFL3718X115, F.Cu at (200.1, 164.7)
- added D_UV6: BAT54T1G, Regen_braking:SODFL3718X115, F.Cu at (158.2, 148.4)
- added D_UV7: BAT54T1G, Regen_braking:SODFL3718X115, F.Cu at (209.7, 45.2)
- added F1: 4628, Regen_braking:FUSE_4628, F.Cu at (271.7, 65.0)
- added IC4: UCC27710DR, Regen_braking:UCC27710DR, B.Cu at (233.0, 94.5)
- added IC5: LM339DT, Regen_braking:SOIC127P600X175-14N, F.Cu at (148.3, 161.1)
- added INOUT_A1: ~, Regen_braking:ACS_pad, F.Cu at (158.4, 140.8)
- added INOUT_B1: ~, Regen_braking:ACS_pad, F.Cu at (24.0, 135.4)
- added J1: XT60PB-M, Regen_braking:XT60PBM, F.Cu at (271.7, 83.1)
- added J10: COMP_EXTI, Connector_PinHeader_2.54mm:PinHeader_1x06_P2.54mm_Vertical, F.Cu at (117.1, 38.3)
- added J11: Conn_01x02, Connector_PinHeader_2.54mm:PinHeader_1x02_P2.54mm_Vertical, F.Cu at (134.6, 74.3)
- added J12: U_ADC, Connector_PinHeader_2.54mm:PinHeader_1x01_P2.54mm_Vertical, F.Cu at (48.6, 117.6)
- added J13: 12V, Connector_Wire:SolderWirePad_1x01_SMD_1.5x3mm, F.Cu at (193.1, 53.3)
- added J14: MOTOR_UVW, Regen_braking:CUI_TB004-508-03BE, F.Cu at (260.8, 165.2)
- added J15: U, Connector_Wire:SolderWirePad_1x01_SMD_1.5x3mm, F.Cu at (207.5, 127.2)
- added J16: BUS, Connector_Wire:SolderWirePad_1x01_SMD_1.5x3mm, F.Cu at (199.7, 45.9)
- added J17: Conn_01x03, Regen_braking:Hall_UVW, F.Cu at (253.8, 153.3)
- added J18: V, Connector_Wire:SolderWirePad_1x01_SMD_1.5x3mm, F.Cu at (240.0, 127.3)
- added J19: W, Connector_Wire:SolderWirePad_1x01_SMD_1.5x3mm, F.Cu at (272.2, 127.3)
- added J2: Conn_01x01, Connector_PinHeader_2.54mm:PinHeader_1x01_P2.54mm_Vertical, F.Cu at (18.0, 23.9)
- added J20: 3V3, Connector_PinHeader_2.54mm:PinHeader_1x01_P2.54mm_Vertical, F.Cu at (68.1, 59.1)
- added J21: ACS1, Connector_PinHeader_2.54mm:PinHeader_1x03_P2.54mm_Vertical, F.Cu at (50.2, 57.4)
- added J22: ACS2, Connector_PinHeader_2.54mm:PinHeader_1x03_P2.54mm_Vertical, F.Cu at (56.6, 57.7)
- added J23: BUS, Connector_Wire:SolderWirePad_1x01_SMD_1.5x3mm, F.Cu at (236.3, 45.6)
- added J24: V_PWM, Connector_PinHeader_2.54mm:PinHeader_1x02_P2.54mm_Vertical, F.Cu at (63.8, 125.0)
- added J25: W_PWM, Connector_PinHeader_2.54mm:PinHeader_1x02_P2.54mm_Vertical, F.Cu at (69.2, 125.0)
- added J26: U_PWM, Connector_PinHeader_2.54mm:PinHeader_1x02_P2.54mm_Vertical, F.Cu at (78.0, 124.3)
- added J27: V_ADC, Connector_PinHeader_2.54mm:PinHeader_1x01_P2.54mm_Vertical, F.Cu at (64.6, 111.3)
- added J28: W_ADC, Connector_PinHeader_2.54mm:PinHeader_1x01_P2.54mm_Vertical, F.Cu at (62.2, 118.3)
- added J29: BAT_ADC, Connector_PinHeader_2.54mm:PinHeader_1x01_P2.54mm_Vertical, F.Cu at (72.5, 107.8)
- added J3: Conn_01x01, Connector_Wire:SolderWirePad_1x01_SMD_1.5x3mm, F.Cu at (22.6, 23.9)
- added J30: CAP_ADC, Connector_PinHeader_2.54mm:PinHeader_1x01_P2.54mm_Vertical, F.Cu at (72.1, 115.0)
- added J31: ACS1_ADC, Connector_PinHeader_2.54mm:PinHeader_1x01_P2.54mm_Vertical, F.Cu at (79.3, 112.6)
- added J32: ACS2_ADC, Connector_PinHeader_2.54mm:PinHeader_1x01_P2.54mm_Vertical, F.Cu at (84.6, 118.1)
- added J4: L_in, Connector_Wire:SolderWirePad_1x01_SMD_1.5x3mm, F.Cu at (149.9, 119.1)
- added J5: 3V3_ports, Connector_PinHeader_2.54mm:PinHeader_1x06_P2.54mm_Vertical, F.Cu at (42.0, 6.94)
- added J6: 5V_ports, Connector_PinHeader_2.54mm:PinHeader_1x06_P2.54mm_Vertical, F.Cu at (27.2, 23.9)
- added J7: GND_ports, Connector_PinHeader_2.54mm:PinHeader_1x10_P2.54mm_Vertical, F.Cu at (112.5, 38.3)
- added J8: GPIO_ports, Connector_PinHeader_2.54mm:PinHeader_1x04_P2.54mm_Vertical, F.Cu at (46.5, 6.94)
- added J9: HALL_EXTI, Connector_PinHeader_2.54mm:PinHeader_1x03_P2.54mm_Vertical, F.Cu at (51.1, 6.95)
- added KCD3-101N1: ~, Regen_braking:Switch_Rocker_KCD3-101N, F.Cu at (259.7, 43.3)
- added L1: 47uH, Regen_braking:CDRH8D43NP220NC, F.Cu at (150.4, 65.4)
- added L2: 33uh, Regen_braking:L_bdc, F.Cu at (149.9, 124.1)
- added NT1: NetTie_2, NetTie:NetTie-2_SMD_Pad2.0mm, F.Cu at (75.3, 91.6)
- added NT2: NetTie_4_Cross, NetTie:NetTie-4_SMD_Pad2.0mm, F.Cu at (163.8, 97.5)
- added NT3: NetTie_4_Cross, NetTie:NetTie-4_SMD_Pad2.0mm, F.Cu at (192.9, 97.5)
- added NT4: NetTie_4_Cross, NetTie:NetTie-4_SMD_Pad2.0mm, F.Cu at (220.0, 97.5)
- added NT5: NetTie_4_Cross, NetTie:NetTie-4_SMD_Pad2.0mm, F.Cu at (246.8, 97.5)
- added Q7: ~, Regen_braking:IRLR3705ZPBF, F.Cu at (246.8, 86.9)
- added Q8: ~, Regen_braking:IRLR3705ZPBF, F.Cu at (247.0, 108.1)
- added R10: 10, Resistor_THT:R_Axial_DIN0207_L6.3mm_D2.5mm_P7.62mm_Horizontal, B.Cu at (149.2, 99.2)
- added R11: 4.7, Resistor_THT:R_Axial_DIN0207_L6.3mm_D2.5mm_P7.62mm_Horizontal, B.Cu at (146.2, 99.2)
- added R12: 22, Resistor_THT:R_Axial_DIN0204_L3.6mm_D1.6mm_P7.62mm_Horizontal, F.Cu at (17.2, 6.77)
- added R13: 22, Resistor_THT:R_Axial_DIN0204_L3.6mm_D1.6mm_P7.62mm_Horizontal, F.Cu at (17.2, 11.0)
- added R14: 22, Resistor_THT:R_Axial_DIN0204_L3.6mm_D1.6mm_P7.62mm_Horizontal, F.Cu at (17.2, 15.3)
- added R15: 22, Resistor_THT:R_Axial_DIN0204_L3.6mm_D1.6mm_P7.62mm_Horizontal, F.Cu at (17.2, 19.5)
- added R16: 10k, Resistor_THT:R_Axial_DIN0204_L3.6mm_D1.6mm_P7.62mm_Horizontal, B.Cu at (182.3, 83.4)
- added R17: 22ohm_snubber, Resistor_THT:R_Axial_DIN0204_L3.6mm_D1.6mm_P7.62mm_Horizontal, B.Cu at (198.0, 81.1)
- added R18: 2.2, Resistor_THT:R_Axial_DIN0207_L6.3mm_D2.5mm_P7.62mm_Horizontal, B.Cu at (185.1, 91.3)
- added R19: 4.7, Resistor_THT:R_Axial_DIN0207_L6.3mm_D2.5mm_P7.62mm_Horizontal, B.Cu at (176.4, 75.7)
- added R20: 47, Resistor_THT:R_Axial_DIN0204_L3.6mm_D1.6mm_P7.62mm_Horizontal, F.Cu at (18.7, 155.4)
- added R21: 10, Resistor_THT:R_Axial_DIN0207_L6.3mm_D2.5mm_P7.62mm_Horizontal, B.Cu at (179.6, 75.7)
- added R22: 22ohm_snubber, Resistor_THT:R_Axial_DIN0204_L3.6mm_D1.6mm_P7.62mm_Horizontal, B.Cu at (198.1, 95.5)
- added R23: 10k, Resistor_THT:R_Axial_DIN0204_L3.6mm_D1.6mm_P7.62mm_Horizontal, B.Cu at (181.2, 106.7)
- added R24: 47, Resistor_THT:R_Axial_DIN0204_L3.6mm_D1.6mm_P7.62mm_Horizontal, F.Cu at (37.1, 155.4)
- added R25: 10, Resistor_THT:R_Axial_DIN0207_L6.3mm_D2.5mm_P7.62mm_Horizontal, B.Cu at (178.5, 99.1)
- added R26: 4.7, Resistor_THT:R_Axial_DIN0207_L6.3mm_D2.5mm_P7.62mm_Horizontal, B.Cu at (175.3, 99.1)
- added R27: 10k, Resistor_THT:R_Axial_DIN0204_L3.6mm_D1.6mm_P7.62mm_Horizontal, B.Cu at (211.5, 83.4)
- added R28: 22ohm_snubber, Resistor_THT:R_Axial_DIN0204_L3.6mm_D1.6mm_P7.62mm_Horizontal, B.Cu at (224.9, 81.1)
- added R29: 2.2, Resistor_THT:R_Axial_DIN0207_L6.3mm_D2.5mm_P7.62mm_Horizontal, B.Cu at (214.3, 91.1)
- added R30: 4.7, Resistor_THT:R_Axial_DIN0207_L6.3mm_D2.5mm_P7.62mm_Horizontal, B.Cu at (205.7, 75.6)
- added R31: 47, Resistor_THT:R_Axial_DIN0204_L3.6mm_D1.6mm_P7.62mm_Horizontal, F.Cu at (18.7, 163.6)
- added R32: 10, Resistor_THT:R_Axial_DIN0207_L6.3mm_D2.5mm_P7.62mm_Horizontal, B.Cu at (208.8, 75.6)
- added R33: 22ohm_snubber, Resistor_THT:R_Axial_DIN0204_L3.6mm_D1.6mm_P7.62mm_Horizontal, B.Cu at (224.9, 95.5)
- added R34: 10k, Resistor_THT:R_Axial_DIN0204_L3.6mm_D1.6mm_P7.62mm_Horizontal, B.Cu at (208.8, 106.8)
- added R35: 47, Resistor_THT:R_Axial_DIN0204_L3.6mm_D1.6mm_P7.62mm_Horizontal, F.Cu at (37.1, 163.6)
- added R36: 10, Resistor_THT:R_Axial_DIN0207_L6.3mm_D2.5mm_P7.62mm_Horizontal, B.Cu at (206.1, 99.3)
- added R37: 4.7, Resistor_THT:R_Axial_DIN0207_L6.3mm_D2.5mm_P7.62mm_Horizontal, B.Cu at (203.0, 99.3)
- added R38: 10k, Resistor_THT:R_Axial_DIN0204_L3.6mm_D1.6mm_P7.62mm_Horizontal, B.Cu at (236.5, 83.2)
- added R39: 2.2, Resistor_THT:R_Axial_DIN0207_L6.3mm_D2.5mm_P7.62mm_Horizontal, B.Cu at (239.8, 91.1)
- added R40: 4.7, Resistor_THT:R_Axial_DIN0207_L6.3mm_D2.5mm_P7.62mm_Horizontal, B.Cu at (230.5, 75.5)
- added R41: 22ohm_snubber, Resistor_THT:R_Axial_DIN0204_L3.6mm_D1.6mm_P7.62mm_Horizontal, B.Cu at (252.4, 80.8)
- added R42: 47, Resistor_THT:R_Axial_DIN0204_L3.6mm_D1.6mm_P7.62mm_Horizontal, F.Cu at (18.7, 171.7)
- added R43: 10, Resistor_THT:R_Axial_DIN0207_L6.3mm_D2.5mm_P7.62mm_Horizontal, B.Cu at (233.7, 75.5)
- added R44: 22ohm_snubber, Resistor_THT:R_Axial_DIN0204_L3.6mm_D1.6mm_P7.62mm_Horizontal, B.Cu at (252.3, 95.3)
- added R45: 10k, Resistor_THT:R_Axial_DIN0204_L3.6mm_D1.6mm_P7.62mm_Horizontal, B.Cu at (235.2, 106.6)
- added R46: 47, Resistor_THT:R_Axial_DIN0204_L3.6mm_D1.6mm_P7.62mm_Horizontal, F.Cu at (37.1, 171.7)
- added R47: 10, Resistor_THT:R_Axial_DIN0207_L6.3mm_D2.5mm_P7.62mm_Horizontal, B.Cu at (232.4, 99.1)
- added R48: 4.7, Resistor_THT:R_Axial_DIN0207_L6.3mm_D2.5mm_P7.62mm_Horizontal, B.Cu at (229.2, 99.1)
- added R49: 10k, Resistor_THT:R_Axial_DIN0204_L3.6mm_D1.6mm_P7.62mm_Horizontal, F.Cu at (245.7, 146.0)
- added R50: 1k, Resistor_THT:R_Axial_DIN0204_L3.6mm_D1.6mm_P7.62mm_Horizontal, F.Cu at (243.5, 138.3)
- added R51: 100k, Resistor_THT:R_Axial_DIN0207_L6.3mm_D2.5mm_P7.62mm_Horizontal, F.Cu at (205.4, 127.5)
- added R52: 1k, Resistor_THT:R_Axial_DIN0204_L3.6mm_D1.6mm_P7.62mm_Horizontal, F.Cu at (195.7, 127.9)
- added R53: 100k, Resistor_THT:R_Axial_DIN0207_L6.3mm_D2.5mm_P7.62mm_Horizontal, F.Cu at (197.5, 46.2)
- added R54: 4.7k, Resistor_THT:R_Axial_DIN0204_L3.6mm_D1.6mm_P7.62mm_Horizontal, F.Cu at (187.8, 46.6)
- added R55: 10k, Resistor_THT:R_Axial_DIN0204_L3.6mm_D1.6mm_P7.62mm_Horizontal, F.Cu at (187.8, 44.4)
- added R56: 10k, Resistor_THT:R_Axial_DIN0204_L3.6mm_D1.6mm_P7.62mm_Horizontal, F.Cu at (195.7, 125.6)
- added R57: 10k, Resistor_THT:R_Axial_DIN0204_L3.6mm_D1.6mm_P7.62mm_Horizontal, F.Cu at (257.1, 146.0)
- added R58: 1k, Resistor_THT:R_Axial_DIN0204_L3.6mm_D1.6mm_P7.62mm_Horizontal, F.Cu at (254.8, 138.4)
- added R59: 10k, Resistor_THT:R_Axial_DIN0204_L3.6mm_D1.6mm_P7.62mm_Horizontal, F.Cu at (143.1, 155.9)
- added R60: 10k, Resistor_THT:R_Axial_DIN0204_L3.6mm_D1.6mm_P7.62mm_Horizontal, F.Cu at (153.6, 158.2)
- added R61: 10k, Resistor_THT:R_Axial_DIN0204_L3.6mm_D1.6mm_P7.62mm_Horizontal, F.Cu at (268.3, 146.0)
- added R62: 100k, Resistor_THT:R_Axial_DIN0207_L6.3mm_D2.5mm_P7.62mm_Horizontal, F.Cu at (237.9, 127.5)
- added R63: 1k, Resistor_THT:R_Axial_DIN0204_L3.6mm_D1.6mm_P7.62mm_Horizontal, F.Cu at (228.1, 128.0)
- added R64: 1k, Resistor_THT:R_Axial_DIN0204_L3.6mm_D1.6mm_P7.62mm_Horizontal, F.Cu at (266.1, 138.4)
- added R65: 10k, Resistor_THT:R_Axial_DIN0204_L3.6mm_D1.6mm_P7.62mm_Horizontal, F.Cu at (228.1, 125.8)
- added R66: 10k, Resistor_THT:R_Axial_DIN0204_L3.6mm_D1.6mm_P7.62mm_Horizontal, F.Cu at (143.1, 158.1)
- added R67: 10k, Resistor_THT:R_Axial_DIN0204_L3.6mm_D1.6mm_P7.62mm_Horizontal, F.Cu at (153.6, 156.0)
- added R68: 100k, Resistor_THT:R_Axial_DIN0207_L6.3mm_D2.5mm_P7.62mm_Horizontal, F.Cu at (270.1, 127.5)
- added R69: 10k, Resistor_THT:R_Axial_DIN0204_L3.6mm_D1.6mm_P7.62mm_Horizontal, F.Cu at (260.4, 125.8)
- added R70: 1k, Resistor_THT:R_Axial_DIN0204_L3.6mm_D1.6mm_P7.62mm_Horizontal, F.Cu at (260.4, 128.0)
- added R71: 100k, Resistor_THT:R_Axial_DIN0207_L6.3mm_D2.5mm_P7.62mm_Horizontal, F.Cu at (178.3, 165.4)
- added R72: 4.7k, Resistor_THT:R_Axial_DIN0204_L3.6mm_D1.6mm_P7.62mm_Horizontal, F.Cu at (188.0, 165.8)
- added R73: 10k, Resistor_THT:R_Axial_DIN0204_L3.6mm_D1.6mm_P7.62mm_Horizontal, F.Cu at (188.0, 163.7)
- added R74: 1k, Resistor_THT:R_Axial_DIN0204_L3.6mm_D1.6mm_P7.62mm_Horizontal, F.Cu at (136.4, 149.5)
- added R75: 4.7k, Resistor_THT:R_Axial_DIN0204_L3.6mm_D1.6mm_P7.62mm_Horizontal, F.Cu at (146.0, 149.5)
- added R76: 2.2k, Resistor_THT:R_Axial_DIN0207_L6.3mm_D2.5mm_P7.62mm_Horizontal, F.Cu at (153.5, 146.8)
- added R77: 220K, Resistor_THT:R_Axial_DIN0207_L6.3mm_D2.5mm_P10.16mm_Horizontal, F.Cu at (234.1, 45.8)
- added R78: 4.7k, Resistor_THT:R_Axial_DIN0204_L3.6mm_D1.6mm_P7.62mm_Horizontal, F.Cu at (221.8, 46.3)
- added R79: 10k, Resistor_THT:R_Axial_DIN0204_L3.6mm_D1.6mm_P7.62mm_Horizontal, F.Cu at (221.8, 44.0)
- added Rbias1: 10, Resistor_THT:R_Axial_DIN0207_L6.3mm_D2.5mm_P7.62mm_Horizontal, F.Cu at (192.0, 57.4)
- added Rbias2: 10, Resistor_THT:R_Axial_DIN0207_L6.3mm_D2.5mm_P7.62mm_Horizontal, F.Cu at (195.1, 57.4)
- added Rbias3: 10, Resistor_THT:R_Axial_DIN0207_L6.3mm_D2.5mm_P7.62mm_Horizontal, F.Cu at (198.2, 57.4)
- added Rbias4: 10, Resistor_THT:R_Axial_DIN0207_L6.3mm_D2.5mm_P7.62mm_Horizontal, F.Cu at (188.8, 57.4)
- added VR1: LM2596S-5.0, Regen_braking:5v_buck, F.Cu at (153.3, 54.9)
- C1: value 4.7uf_50v_VDDcap -> 330u; footprint Regen_braking:4.7uf_50v_VDDcap -> Capacitor_THT:CP_Radial_D10.0mm_P5.00mm
- C2: value 0.47uf_50v_BScap -> 1u; footprint Regen_braking:0.47uf_50v_BScap -> Capacitor_SMD:C_0805_2012Metric
- C3: value 4.7uf_50v_VDDcap -> 120uf; footprint Regen_braking:4.7uf_50v_VDDcap -> Regen_braking:120uf_cap_5v_buck
- C4, C6: value 0.47uf_50v_BScap -> 1000uf; footprint Regen_braking:0.47uf_50v_BScap -> Capacitor_THT:C_Radial_D12.5mm_H25.0mm_P5.00mm
- C5: value 4.7uf_50v_VDDcap -> 1000uf; footprint Regen_braking:4.7uf_50v_VDDcap -> Capacitor_THT:C_Radial_D12.5mm_H25.0mm_P5.00mm
- D1: value SS34_BootDiode -> SS34; footprint Regen_braking:boot_diode -> Regen_braking:DIO_SS34
- D2: value SS34_BootDiode -> SMBJ33A; footprint Regen_braking:boot_diode -> Regen_braking:DIOM5336X244N
- D3: value SS34_BootDiode -> 1N5822; footprint Regen_braking:boot_diode -> Regen_braking:DIOAD1990W125L900D530
- D4: value SS34_BootDiode -> D_boot; moved to B.Cu
- D5: value SS34_BootDiode -> SS34_H; footprint Regen_braking:boot_diode -> Regen_braking:DIO_SS34; moved to B.Cu
- D6: value SS34_BootDiode -> SS34_L; footprint Regen_braking:boot_diode -> Regen_braking:DIO_SS34; moved to B.Cu
- D7, D8, D9: value SS34_BootDiode -> LED; footprint Regen_braking:boot_diode -> LED_THT:LED_D5.0mm
- IC1, IC2, IC3: value IRS21867STRPBF -> UCC27710DR; footprint Regen_braking:IRS21867STRPBF_gatedriver -> Regen_braking:UCC27710DR; moved to B.Cu
- R1: value Rboot_22ohm -> 10k; footprint Regen_braking:Rboot_22ohm -> Resistor_THT:R_Axial_DIN0204_L3.6mm_D1.6mm_P7.62mm_Horizontal; moved to B.Cu
- R2: value R_OFF_5.1ohm -> 22ohm_snubber; footprint Regen_braking:R_OFF_5.1ohm -> Resistor_THT:R_Axial_DIN0204_L3.6mm_D1.6mm_P7.62mm_Horizontal; moved to B.Cu
- R3: value R_OFF_5.1ohm -> 2.2; footprint Regen_braking:R_OFF_5.1ohm -> Resistor_THT:R_Axial_DIN0207_L6.3mm_D2.5mm_P7.62mm_Horizontal; moved to B.Cu
- R4: value Rboot_22ohm -> 4.7; footprint Regen_braking:Rboot_22ohm -> Resistor_THT:R_Axial_DIN0207_L6.3mm_D2.5mm_P7.62mm_Horizontal; moved to B.Cu
- R5, R9: value R_OFF_5.1ohm -> 47; footprint Regen_braking:R_OFF_5.1ohm -> Resistor_THT:R_Axial_DIN0204_L3.6mm_D1.6mm_P7.62mm_Horizontal
- R6: value R_OFF_5.1ohm -> 10; footprint Regen_braking:R_OFF_5.1ohm -> Resistor_THT:R_Axial_DIN0207_L6.3mm_D2.5mm_P7.62mm_Horizontal; moved to B.Cu
- R7: value Rboot_22ohm -> 22ohm_snubber; footprint Regen_braking:Rboot_22ohm -> Resistor_THT:R_Axial_DIN0204_L3.6mm_D1.6mm_P7.62mm_Horizontal; moved to B.Cu
- R8: value R_OFF_5.1ohm -> 10k; footprint Regen_braking:R_OFF_5.1ohm -> Resistor_THT:R_Axial_DIN0204_L3.6mm_D1.6mm_P7.62mm_Horizontal; moved to B.Cu
- moved R5 173.2 mm to (18.7, 178.7)
- moved R9 152.8 mm to (37.1, 178.7), turned to 180 degrees
- moved D2 142.8 mm to (264.2, 56.4), turned to -90 degrees
- moved C2 137.4 mm to (260.8, 54.6), turned to -90 degrees
- moved C1 136.2 mm to (254.8, 55.3), turned to -90 degrees
- moved D1 122.0 mm to (243.8, 56.0)
- moved Q5 101.2 mm to (219.8, 86.9), turned to 90 degrees
- moved Q6 98.1 mm to (220.0, 108.1), turned to 90 degrees
- moved IC3 75.2 mm to (207.5, 94.5), turned to 180 degrees
- moved Q3 70.9 mm to (192.8, 86.9), turned to 90 degrees
- moved Q4 69.5 mm to (193.0, 108.1), turned to 90 degrees
- moved D7 69.3 mm to (95.2, 13.7)
- moved D8 69.3 mm to (95.2, 21.2)
- moved D9 69.3 mm to (95.2, 28.6)
- moved C3 69.1 mm to (166.4, 59.0), turned to 90 degrees
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Connections:
- C1 pad 1: /Inverter Stage/Vcc_15v -> Net-(D2-K)
- C1 pad 2: GND -> 0
- C2 pad 1: /Inverter Stage/VB_1 -> Net-(D2-K)
- C2 pad 2: /Inverter Stage/VS_1 -> 0
- C4 pad 1: /Inverter Stage/VB_2 -> /Battery & Super Capacitor Buffer/Cap_bufferBank
- C4 pad 2: /Inverter Stage/VS_2 -> 0
- C5 pad 1: /Inverter Stage/Vcc_15v -> /Battery & Super Capacitor Buffer/Cap_bufferBank
- C5 pad 2: GND -> 0
- C6 pad 1: /Inverter Stage/VB_3 -> /Battery & Super Capacitor Buffer/Cap_bufferBank
- C6 pad 2: /Inverter Stage/VS_3 -> 0
- D1 pad A: Net-(D1-PadA) -> Net-(D2-K)
- D1 pad C: /Inverter Stage/VB_1 -> /Battery & Super Capacitor Buffer/DC_BUS
- D3 pad A: /Inverter Stage/GL1 -> 0
- D3 pad C: Net-(D3-PadC) -> /Battery & Super Capacitor Buffer/SW
- D5 pad A: /Inverter Stage/GH2 -> /Battery & Super Capacitor Buffer/GH
- D6 pad A: /Inverter Stage/GL2 -> /Battery & Super Capacitor Buffer/GL
- IC1 pad 1: /Inverter Stage/Vcc_15v -> /Battery & Super Capacitor Buffer/VDD
- IC1 pad 2: /Inverter Stage/U_HIN -> /Battery & Super Capacitor Buffer/HIN
- IC1 pad 3: /Inverter Stage/U_LIN -> /Battery & Super Capacitor Buffer/LIN
- IC1 pad 4: GND -> 0
- IC1 pad 5: /Inverter Stage/U_LOUT -> /Battery & Super Capacitor Buffer/QL_out
- IC1 pad 6: /Inverter Stage/VS_1 -> /Battery & Super Capacitor Buffer/VS
- IC1 pad 7: /Inverter Stage/U_HOUT -> /Battery & Super Capacitor Buffer/QH_out
- IC1 pad 8: /Inverter Stage/VB_1 -> /Battery & Super Capacitor Buffer/VB
- IC2 pad 1: /Inverter Stage/Vcc_15v -> /Inverter Stage/Vcc_12v_1
- IC2 pad 2: /Inverter Stage/V_HIN -> /Inverter Stage/U_HIN
- IC2 pad 3: /Inverter Stage/V_LIN -> /Inverter Stage/U_LIN
- IC2 pad 4: GND -> 0
- IC2 pad 5: /Inverter Stage/V_LOUT -> /Inverter Stage/U_LOUT
- IC2 pad 6: /Inverter Stage/VS_2 -> /Inverter Stage/VS_1
- IC2 pad 7: /Inverter Stage/V_HOUT -> /Inverter Stage/U_HOUT
- IC2 pad 8: /Inverter Stage/VB_2 -> /Inverter Stage/VB_1
- IC3 pad 1: /Inverter Stage/Vcc_15v -> /Inverter Stage/Vcc_12v_2
- IC3 pad 2: /Inverter Stage/W_HIN -> /Inverter Stage/V_HIN
- IC3 pad 3: /Inverter Stage/W_LIN -> /Inverter Stage/V_LIN
- IC3 pad 4: GND -> 0
- IC3 pad 5: /Inverter Stage/W_LOUT -> /Inverter Stage/V_LOUT
- IC3 pad 6: /Inverter Stage/VS_3 -> /Inverter Stage/VS_2
- IC3 pad 7: /Inverter Stage/W_HOUT -> /Inverter Stage/V_HOUT
- IC3 pad 8: /Inverter Stage/VB_3 -> /Inverter Stage/VB_2
- Q1 pad 1: /Inverter Stage/GH1 -> /Battery & Super Capacitor Buffer/GH
- Q1 pad 3: /Inverter Stage/VS_1 -> Net-(Q1-S)
- Q2 pad 1: /Inverter Stage/GL1 -> /Battery & Super Capacitor Buffer/GL
- Q2 pad 3: unconnected-(Q2-S-Pad3) -> 0
- Q3 pad 1: /Inverter Stage/GH2 -> /Inverter Stage/GH1
- Q3 pad 3: /Inverter Stage/VS_1 -> Net-(Q3-S)
- Q4 pad 1: /Inverter Stage/GL2 -> /Inverter Stage/GL1
- Q4 pad 3: unconnected-(Q4-S-Pad3) -> 0
- Q5 pad 1: /Inverter Stage/GH3 -> /Inverter Stage/GH2
- Q5 pad 3: /Inverter Stage/VS_1 -> Net-(Q5-S)
- Q6 pad 1: /Inverter Stage/GL3 -> /Inverter Stage/GL2
- Q6 pad 3: unconnected-(Q6-S-Pad3) -> 0
- R1 pad 1: /Inverter Stage/Vcc_15v -> /Battery & Super Capacitor Buffer/GH
- R1 pad 2: Net-(D1-PadA) -> /Battery & Super Capacitor Buffer/VS
- R2 pad 1: /Inverter Stage/U_HOUT -> /Battery & Super Capacitor Buffer/VBUS
- R2 pad 2: Net-(D2-PadC) -> Net-(C16-Pad1)
- R3 pad 1: /Inverter Stage/U_LOUT -> /Battery & Super Capacitor Buffer/VDD
- R3 pad 2: Net-(D3-PadC) -> Net-(D4-A)
- R4 pad 1: /Inverter Stage/Vcc_15v -> /Battery & Super Capacitor Buffer/QH_out
- R4 pad 2: Net-(D4-PadA) -> Net-(D5-PadC)
- R5 pad 1: /Inverter Stage/U_HOUT -> /Battery & Super Capacitor Buffer/Q_HIGH
- R5 pad 2: Net-(D5-PadC) -> /Battery & Super Capacitor Buffer/HIN
- R6 pad 1: /Inverter Stage/V_LOUT -> /Battery & Super Capacitor Buffer/QH_out
- R6 pad 2: Net-(D6-PadC) -> /Battery & Super Capacitor Buffer/GH
- R7 pad 1: /Inverter Stage/Vcc_15v -> /Battery & Super Capacitor Buffer/VS
- R7 pad 2: Net-(D7-PadA) -> Net-(C18-Pad1)
- R8 pad 1: /Inverter Stage/W_HOUT -> /Battery & Super Capacitor Buffer/GL
- R8 pad 2: Net-(D8-PadC) -> 0
- R9 pad 1: /Inverter Stage/W_LOUT -> /Battery & Super Capacitor Buffer/Q_LOW
- R9 pad 2: Net-(D9-PadC) -> /Battery & Super Capacitor Buffer/LIN
Routing:
- added copper zone on In1.Cu, net 0
Other:
- board outline added: 150 x 150 mm
- copper layers 2 -> 4

Commit message: ------------------Project Completed Successfully------------------
Parts:
- removed J16: BUS, Connector_Wire:SolderWirePad_1x01_SMD_1.5x3mm
- removed J22: ACS2, Connector_PinHeader_2.54mm:PinHeader_1x03_P2.54mm_Vertical
- removed J3: Conn_01x01, Connector_Wire:SolderWirePad_1x01_SMD_1.5x3mm
- removed J31: ACS1_ADC, Connector_PinHeader_2.54mm:PinHeader_1x01_P2.54mm_Vertical
- removed J32: ACS2_ADC, Connector_PinHeader_2.54mm:PinHeader_1x01_P2.54mm_Vertical
- J11: value Conn_01x02 -> U_PWM
- J17: value Conn_01x03 -> HALL_EXTI
- J2: value Conn_01x01 -> 5V
- J21: value ACS1 -> ACS1_ADC; footprint Connector_PinHeader_2.54mm:PinHeader_1x03_P2.54mm_Vertical -> Connector_PinHeader_2.54mm:PinHeader_1x01_P2.54mm_Vertical
- J26: value U_PWM -> Q_PWM
- Rbias1, Rbias2, Rbias3, Rbias4: moved to B.Cu
- moved J9 168.1 mm to (168.9, 127.0), turned to 90 degrees
- moved C47 162.8 mm to (93.6, 156.8)
- moved J23 162.8 mm to (117.9, 157.3)
- moved R77 162.8 mm to (115.7, 157.6)
- moved R78 162.8 mm to (103.4, 158.0)
- moved D_OV7 162.8 mm to (89.1, 156.8)
- moved D_UV7 162.8 mm to (91.3, 157.0)
- moved R79 162.8 mm to (103.4, 155.8)
- moved R42 160.7 mm to (148.4, 76.7), turned to -90 degrees
- moved C31 153.6 mm to (152.8, 87.6)
- moved C35 152.0 mm to (154.8, 89.0), turned to 90 degrees
- moved INOUT_B1 148.7 mm to (138.5, 40.5), turned to 180 degrees
- moved R31 132.6 mm to (118.5, 76.3), turned to -90 degrees
- moved R46 131.7 mm to (147.6, 99.8), turned to 90 degrees
- moved J10 126.9 mm to (72.2, 156.9), turned to 90 degrees
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Connections:
- net /Battery & Super Capacitor Buffer/Cap_bufferBank renamed Cap_bufferBank
- net /Inverter Stage/12V renamed 12V
- net /Inverter Stage/Vcc_12v_1 renamed Vcc_12v_1
- net /Inverter Stage/Vcc_12v_2 renamed Vcc_12v_2
- net /Inverter Stage/Vcc_12v_3 renamed Vcc_12v_3
- net /Sensors/3V3 renamed 3V3
- net /Sensors/OC_mid renamed OC_mid
- net /Sensors/REF renamed REF
- C1 pad 2: 0 -> GND
- C10 pad 2: 0 -> GND
- C11 pad 2: 0 -> GND
- C12 pad 2: 0 -> GND
- C13 pad 2: 0 -> GND
- C14 pad 2: 0 -> GND
- C17 pad 1: /Battery & Super Capacitor Buffer/VDD -> VDD
- C17 pad 2: 0 -> GND
- C18 pad 2: 0 -> GND
- C2 pad 2: 0 -> GND
- C20 pad 2: 0 -> GND
- C22 pad 2: 0 -> GND
- C23 pad 2: 0 -> GND
- C24 pad 2: 0 -> GND
- C26 pad 2: 0 -> GND
- C28 pad 2: 0 -> GND
- C29 pad 2: 0 -> GND
- C3 pad N: 0 -> GND
- C3 pad P: /Battery & Super Capacitor Buffer/VBUS -> VBUS
- C30 pad 2: 0 -> GND
- C31 pad 2: 0 -> GND
- C34 pad 2: 0 -> GND
- C35 pad 2: 0 -> GND
- C36 pad 2: 0 -> GND
- C37 pad 1: /Sensors/Hall_U -> Hall_U
- C38 pad 1: /Sensors/U_ADC1 -> U_ADC1
- C39 pad 1: /Sensors/VSENSE_BAT -> VSENSE_BAT
- C4 pad 2: 0 -> GND
- C40 pad 1: /Sensors/Hall_V -> Hall_V
- C41 pad 1: /Sensors/5V -> 5V
- C41 pad 2: /Sensors/GND -> GND
- C42 pad 1: /Sensors/V_ADC1 -> V_ADC1
- C43 pad 1: /Sensors/Hall_W -> Hall_W
- C44 pad 1: /Sensors/W_ADC1 -> W_ADC1
- C45 pad 1: /Sensors/VSENSE_CAP -> VSENSE_CAP
- C5 pad 2: 0 -> GND
- C6 pad 2: 0 -> GND
- C7 pad 2: 0 -> GND
- C8 pad 2: 0 -> GND
- C9 pad 1: /Battery & Super Capacitor Buffer/5V -> 5V
- C9 pad 2: 0 -> GND
- C_Hi1 pad 2: 0 -> GND
- C_Li1 pad 2: 0 -> GND
- D1 pad C: /Battery & Super Capacitor Buffer/DC_BUS -> DC_BUS
- D10 pad 1: /MCU & Peripherals/GND -> GND
- D2 pad 2: 0 -> GND
- D3 pad A: 0 -> GND
- D7 pad 1: /MCU & Peripherals/GND -> GND
- D8 pad 1: /MCU & Peripherals/GND -> GND
- D9 pad 1: /MCU & Peripherals/GND -> GND
- D_OV1 pad 1: /Sensors/VSENSE_BAT -> VSENSE_BAT
- D_OV2 pad 1: /Sensors/U_ADC1 -> U_ADC1
- D_OV3 pad 1: /Sensors/V_ADC1 -> V_ADC1
- D_OV4 pad 1: /Sensors/W_ADC1 -> W_ADC1
- D_OV5 pad 1: /Sensors/VSENSE_CAP -> VSENSE_CAP
- D_UV1 pad 2: /Sensors/U_ADC1 -> U_ADC1
- D_UV2 pad 2: /Sensors/VSENSE_BAT -> VSENSE_BAT
- D_UV3 pad 2: /Sensors/V_ADC1 -> V_ADC1
- D_UV4 pad 2: /Sensors/W_ADC1 -> W_ADC1
- D_UV5 pad 2: /Sensors/VSENSE_CAP -> VSENSE_CAP
- IC1 pad 1: /Battery & Super Capacitor Buffer/VDD -> VDD
- IC1 pad 4: 0 -> GND
- IC2 pad 4: 0 -> GND
- IC3 pad 4: 0 -> GND
- IC4 pad 4: 0 -> GND
- IC5 pad 1: /Sensors/OUT2 -> OUT2
- IC5 pad 11: /Sensors/ACS1 -> ACS1
- IC5 pad 12: /Sensors/GND -> GND
- IC5 pad 13: /Sensors/OUT4 -> OUT4
- IC5 pad 14: /Sensors/OUT3 -> OUT3
- IC5 pad 2: /Sensors/OUT1 -> OUT1
- IC5 pad 3: /Sensors/5V -> 5V
- IC5 pad 5: /Sensors/U_ADC1 -> U_ADC1
- IC5 pad 7: /Sensors/V_ADC1 -> V_ADC1
- IC5 pad 9: /Sensors/W_ADC1 -> W_ADC1
- INOUT_A1 pad 1: /Sensors/ACS_in -> ACS_in
- INOUT_B1 pad 1: /Sensors/DC_BUS -> DC_BUS
- INOUT_B1 pad 2: /Sensors/VBUS -> VBUS
- J1 pad 2: 0 -> GND
- J10 pad 1: /MCU & Peripherals/OUT1 -> OUT1
- J10 pad 2: /MCU & Peripherals/OUT2 -> OUT2
- J10 pad 3: /MCU & Peripherals/OUT3 -> OUT3
- J10 pad 4: /MCU & Peripherals/OUT4 -> OUT4
- J10 pad 5: /MCU & Peripherals/OUT4 -> OUT4
- J10 pad 6: /MCU & Peripherals/OUT4 -> OUT4
- J11 pad 1: /MCU & Peripherals/U_HIGH -> U_HIGH
- J11 pad 2: /MCU & Peripherals/U_LOW -> U_LOW
- J12 pad 1: /MCU & Peripherals/U_ADC1 -> U_ADC1
- J2 pad 1: /Battery & Super Capacitor Buffer/5V -> 5V
- J21 pad 1: GNDA -> ACS1
- J24 pad 1: /MCU & Peripherals/V_LOW -> V_LOW
- J24 pad 2: /MCU & Peripherals/V_HIGH -> V_HIGH
- J25 pad 1: /MCU & Peripherals/W_HIGH -> W_HIGH
- J25 pad 2: /MCU & Peripherals/W_LOW -> W_LOW
- J26 pad 1: /MCU & Peripherals/Q_HIGH -> Q_HIGH
- J26 pad 2: /MCU & Peripherals/Q_LOW -> Q_LOW
- J27 pad 1: /MCU & Peripherals/V_ADC1 -> V_ADC1
- J28 pad 1: /MCU & Peripherals/W_ADC1 -> W_ADC1
- J29 pad 1: /MCU & Peripherals/VSENSE_BAT -> VSENSE_BAT
- J30 pad 1: /MCU & Peripherals/VSENSE_CAP -> VSENSE_CAP
- J7 pad 1: /MCU & Peripherals/GND -> GND
- J7 pad 10: /MCU & Peripherals/GND -> GND
- J7 pad 2: /MCU & Peripherals/GND -> GND
- J7 pad 3: /MCU & Peripherals/GND -> GND
- J7 pad 4: /MCU & Peripherals/GND -> GND
- J7 pad 5: /MCU & Peripherals/GND -> GND
- J7 pad 6: /MCU & Peripherals/GND -> GND
- J7 pad 7: /MCU & Peripherals/GND -> GND
- J7 pad 8: /MCU & Peripherals/GND -> GND
- J7 pad 9: /MCU & Peripherals/GND -> GND
- J9 pad 1: /MCU & Peripherals/Hall_U -> Hall_U
- J9 pad 2: /MCU & Peripherals/Hall_V -> Hall_V
- J9 pad 3: /MCU & Peripherals/Hall_W -> Hall_W
- L1 pad 2: /Battery & Super Capacitor Buffer/5V -> 5V
- L2 pad 2: /Battery & Super Capacitor Buffer/ACS_in -> ACS_in
- NT1 pad 2: 0 -> GND
- NT2 pad 2: unconnected-(NT2-Pad2) -> /Battery & Super Capacitor Buffer/VS
- NT2 pad 3: Net-(Q1-S) -> /Battery & Super Capacitor Buffer/VS
- NT2 pad 4: Net-(Q2-D) -> /Battery & Super Capacitor Buffer/VS
- NT3 pad 2: unconnected-(NT3-Pad2) -> /Inverter Stage/VS_1
- NT3 pad 3: Net-(Q3-S) -> /Inverter Stage/VS_1
- NT3 pad 4: Net-(Q4-D) -> /Inverter Stage/VS_1
- NT4 pad 2: unconnected-(NT4-Pad2) -> /Inverter Stage/VS_2
- NT4 pad 3: Net-(Q5-S) -> /Inverter Stage/VS_2
- NT4 pad 4: Net-(Q6-D) -> /Inverter Stage/VS_2
- NT5 pad 2: unconnected-(NT5-Pad2) -> /Inverter Stage/VS_3
- NT5 pad 3: Net-(Q7-S) -> /Inverter Stage/VS_3
- NT5 pad 4: Net-(Q8-D) -> /Inverter Stage/VS_3
- Q1 pad 2: /Battery & Super Capacitor Buffer/VBUS -> VBUS
- Q1 pad 3: Net-(Q1-S) -> /Battery & Super Capacitor Buffer/VS
- Q2 pad 2: Net-(Q2-D) -> /Battery & Super Capacitor Buffer/VS
- Q2 pad 3: 0 -> GND
- Q3 pad 2: /Inverter Stage/VBUS -> VBUS
- Q3 pad 3: Net-(Q3-S) -> /Inverter Stage/VS_1
- Q4 pad 2: Net-(Q4-D) -> /Inverter Stage/VS_1
- Q4 pad 3: 0 -> GND
- Q5 pad 2: /Inverter Stage/VBUS -> VBUS
- Q5 pad 3: Net-(Q5-S) -> /Inverter Stage/VS_2
- Q6 pad 2: Net-(Q6-D) -> /Inverter Stage/VS_2
- Q6 pad 3: 0 -> GND
- Q7 pad 2: /Inverter Stage/VBUS -> VBUS
- Q7 pad 3: Net-(Q7-S) -> /Inverter Stage/VS_3
- Q8 pad 2: Net-(Q8-D) -> /Inverter Stage/VS_3
- Q8 pad 3: 0 -> GND
- R17 pad 1: /Inverter Stage/VBUS -> VBUS
- R2 pad 1: /Battery & Super Capacitor Buffer/VBUS -> VBUS
- R20 pad 1: /Inverter Stage/U_HIGH -> U_HIGH
- R23 pad 2: 0 -> GND
- R24 pad 1: /Inverter Stage/U_LOW -> U_LOW
- R28 pad 1: /Inverter Stage/VBUS -> VBUS
- R3 pad 1: /Battery & Super Capacitor Buffer/VDD -> VDD
- R31 pad 1: /Inverter Stage/V_HIGH -> V_HIGH
- R34 pad 2: 0 -> GND
- R35 pad 1: /Inverter Stage/V_LOW -> V_LOW
- R41 pad 1: /Inverter Stage/VBUS -> VBUS
- R42 pad 1: /Inverter Stage/W_HIGH -> W_HIGH
- R45 pad 2: 0 -> GND
- R46 pad 1: /Inverter Stage/W_LOW -> W_LOW
- R5 pad 1: /Battery & Super Capacitor Buffer/Q_HIGH -> Q_HIGH
- R50 pad 1: /Sensors/Hall_U -> Hall_U
- R52 pad 2: /Sensors/U_ADC1 -> U_ADC1
- R53 pad 1: Net-(J16-Pin_1) -> VBUS
- R54 pad 2: /Sensors/VSENSE_BAT -> VSENSE_BAT
- R58 pad 1: /Sensors/Hall_V -> Hall_V
- R59 pad 1: /Sensors/OUT2 -> OUT2
- R60 pad 1: /Sensors/OUT4 -> OUT4
- R63 pad 2: /Sensors/V_ADC1 -> V_ADC1
- R64 pad 1: /Sensors/Hall_W -> Hall_W
- R66 pad 1: /Sensors/OUT1 -> OUT1
- R67 pad 1: /Sensors/OUT3 -> OUT3
- R70 pad 2: /Sensors/W_ADC1 -> W_ADC1
- R72 pad 2: /Sensors/VSENSE_CAP -> VSENSE_CAP
- R74 pad 1: /Sensors/5V -> 5V
- R8 pad 2: 0 -> GND
- R9 pad 1: /Battery & Super Capacitor Buffer/Q_LOW -> Q_LOW
- Rbias4 pad 2: /Inverter Stage/VDD -> VDD
- VR1 pad 1: /Battery & Super Capacitor Buffer/VBUS -> VBUS
- VR1 pad 3: 0 -> GND
- VR1 pad 4: /Battery & Super Capacitor Buffer/5V -> 5V
- VR1 pad 5: 0 -> GND
- VR1 pad 6: 0 -> GND
Routing:
- net GND: track 0.00 -> 428.0 mm, vias 0 -> 12
- net GNDA: track 0.00 -> 365.3 mm
- net VBUS: track 0.00 -> 224.4 mm, vias 0 -> 1
- net Cap_bufferBank: track 0.00 -> 147.9 mm
- net 5V: track 0.00 -> 140.7 mm
- net W_ADC1: track 0.00 -> 112.5 mm, vias 0 -> 1
- net V_ADC1: track 0.00 -> 86.1 mm, vias 0 -> 1
- net Vcc_12v_3: track 0.00 -> 70.1 mm
- net VDD: track 0.00 -> 69.3 mm
- net U_ADC1: track 0.00 -> 58.8 mm, vias 0 -> 1
- net /Battery & Super Capacitor Buffer/VS: track 0.00 -> 55.8 mm, vias 0 -> 2
- net /Inverter Stage/VS_1: track 0.00 -> 53.8 mm, vias 0 -> 1
- net /Inverter Stage/VS_3: track 0.00 -> 50.7 mm, vias 0 -> 2
- net /Inverter Stage/VS_2: track 0.00 -> 48.3 mm, vias 0 -> 2
- net Vcc_12v_2: track 0.00 -> 40.2 mm
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- added copper zone on F.Cu, net /Battery & Super Capacitor Buffer/VS
- added copper zone on F.Cu, net /Inverter Stage/VS_1
- added copper zone on F.Cu, net /Inverter Stage/VS_2
- added copper zone on F.Cu, net /Inverter Stage/VS_3
- added copper zone on In2.Cu, net 3V3
- added copper zone on In1.Cu, net GND
- removed copper zone on In1.Cu, net 0
Other:
- board size 150 x 150 mm -> 145.8 x 130.1 mm
