File: Hardware/Regenerative_Braking/Sensors.kicad_sch (KiCad schematic)
At the start: 62 parts, among them IC4 LM339DT, J2 Conn_01x03

Commit message: finished placement
Parts:
- removed ACS712-30A1, ACS712-30A4: (no value), Regen_braking:ACS712_Module_27x12mm, symbol Regen_braking:ACS712-30A
- added J15, J16, J18, J19, J23: Conn_01x01, Connector_Wire:SolderWirePad_1x01_SMD_1.5x3mm, symbol Connector_Generic:Conn_01x01
- added J20: Conn_01x01, Connector_PinHeader_2.54mm:PinHeader_1x01_P2.54mm_Vertical, symbol Connector_Generic:Conn_01x01
- added J21, J22: Conn_01x03, Connector_PinHeader_2.54mm:PinHeader_1x03_P2.54mm_Vertical, symbol Connector_Generic:Conn_01x03
- C37: renamed from C36; footprint Capacitor_SMD:C_1206_3216Metric -> Capacitor_THT:C_Disc_D6.0mm_W4.4mm_P5.00mm
- C38: renamed from C7; footprint Capacitor_SMD:C_1206_3216Metric -> Capacitor_THT:C_Disc_D6.0mm_W4.4mm_P5.00mm
- C40: renamed from C37; footprint Capacitor_SMD:C_1206_3216Metric -> Capacitor_THT:C_Disc_D6.0mm_W4.4mm_P5.00mm
- C42: renamed from C8; footprint Capacitor_SMD:C_1206_3216Metric -> Capacitor_THT:C_Disc_D6.0mm_W4.4mm_P5.00mm
- C43: renamed from C38; footprint Capacitor_SMD:C_1206_3216Metric -> Capacitor_THT:C_Disc_D6.0mm_W4.4mm_P5.00mm
- C44: renamed from C9; footprint Capacitor_SMD:C_1206_3216Metric -> Capacitor_THT:C_Disc_D6.0mm_W4.4mm_P5.00mm
- renumbered C40 to C39, C20 to C41, C41 to C45, C19 to C46, C17 to C47, D_OV8 to D_OV1, D_OV1 to D_OV2, D_OV2 to D_OV3, D_OV3 to D_OV4, D_OV10 to D_OV5, D_OV9 to D_OV6, D_OV5 to D_OV7, D_UV8 to D_UV2, D_UV2 to D_UV3, D_UV3 to D_UV4, D_UV10 to D_UV5, D_UV9 to D_UV6, D_UV5 to D_UV7, IC4 to IC5, ACS712-30A3 to INOUT_A1, ACS712-30A2 to INOUT_B1, J2 to J17, R19 to R49, R41 to R50, R1 to R51, R26 to R52, R7 to R53, R29 to R54, R8 to R55, R4 to R56, R30 to R57, R42 to R58, R17 to R59, R18 to R60, R31 to R61, R2 to R62, R27 to R63, R43 to R64, R5 to R65, R20 to R66, R21 to R67, R3 to R68, R6 to R69, R28 to R70, R32 to R71, R34 to R72, R33 to R73, R40 to R74, R36 to R75, R22 to R76, R15 to R77, R25 to R78, R16 to R79
Connections:
- net 3V3: now also J20.1 (Pin_1)
- net 5V: now also J21.3 (Pin_3), J22.3 (Pin_3)
- net ACS1: now also J21.2 (Pin_2)
- net ACS2: now also J22.2 (Pin_2)
- net ACS_in: now also INOUT_A1.1 (IN); no longer INOUT_A1. (OUT)
- net Cap_bufferBank: now also INOUT_A1.2 (OUT); no longer INOUT_A1. (OUT)
- net DC_BUS: now also INOUT_B1.1 (IN); no longer INOUT_B1. (OUT)
- net GND: no longer C37.2, C38.2, C39.2, C40.2, C42.2, C43.2, C44.2, C45.2, C46.2, C47.2, D_UV1.1, D_UV2.1, D_UV3.1, D_UV4.1, D_UV5.1, D_UV6.1, D_UV7.1, R55.2, R56.2, R65.2, R69.2, R73.2, R76.1, R79.2
- net VBUS: now also INOUT_B1.2 (OUT); no longer INOUT_B1. (OUT), R53.1, R77.1
- net Phase_U: no longer names the net of R51.1
- net Phase_U: now also J15.1 (Pin_1)
- net Phase_V: no longer names the net of R62.1
- net Phase_V: now also J18.1 (Pin_1)
- net Phase_W: no longer names the net of R68.1
- net Phase_W: now also J19.1 (Pin_1)
- new net: J16.1 (Pin_1), R53.1
- new net: J23.1 (Pin_1), R77.1
- new net GNDA: C37.2, C38.2, C39.2, C40.2, C42.2, C43.2, C44.2, C45.2, C46.2, C47.2, D_UV1.1, D_UV2.1, D_UV3.1, D_UV4.1, D_UV5.1, D_UV6.1, D_UV7.1, J21.1 (Pin_1), J22.1 (Pin_1), R55.2, R56.2, R65.2, R69.2, R73.2, R76.1, R79.2
Other:
- moved on the sheet: R69

Commit message: ------------------Project Completed Successfully------------------
Parts:
- removed J16: Conn_01x01, Connector_Wire:SolderWirePad_1x01_SMD_1.5x3mm, symbol Connector_Generic:Conn_01x01
- removed J21, J22: Conn_01x03, Connector_PinHeader_2.54mm:PinHeader_1x03_P2.54mm_Vertical, symbol Connector_Generic:Conn_01x03
- J15: value Conn_01x01 -> U
- J17: value Conn_01x03 -> HALL_EXTI
- J18: value Conn_01x01 -> V
- J19: value Conn_01x01 -> W
- J20: value Conn_01x01 -> 3V3
- J23: value Conn_01x01 -> BUS
Connections:
- net VBUS: now also R53.1
Other:
- moved on the sheet: INOUT_B1, J20
